File: 4keymacropad.kicad_pcb (KiCad board)
At the start: 2 copper layers, 78.5 x 41.2 mm, 9 parts, among them J1 Conn_01x05, SW1 SW_Push, SW2 SW_Push, SW3 SW_Push, SW4 SW_Push

Commit message: Updates to use rows/columns from mainboard
Parts:
- added D1: 1N4148W, Diode_SMD:D_SOD-123, B.Cu at (165.5, 100.0)
- added D2: 1N4148W, Diode_SMD:D_SOD-123, B.Cu at (144.1, 98.4)
- added D3: 1N4148W, Diode_SMD:D_SOD-123, B.Cu at (125.0, 98.3)
- added D4: 1N4148W, Diode_SMD:D_SOD-123, B.Cu at (144.0, 79.5)
Connections:
- net GND renamed /ROW2
- J1 pad 2: Net-(J1-Pad2) -> /UP
- J1 pad 3: Net-(J1-Pad3) -> /LEFT
- J1 pad 4: Net-(J1-Pad4) -> /DOWN
- J1 pad 5: Net-(J1-Pad5) -> /RIGHT
- SW1 pad 1: Net-(J1-Pad2) -> Net-(D4-Pad2)
- SW2 pad 1: Net-(J1-Pad3) -> Net-(D3-Pad2)
- SW3 pad 1: Net-(J1-Pad4) -> Net-(D2-Pad2)
- SW4 pad 1: Net-(J1-Pad5) -> Net-(D1-Pad2)
Routing:
- net Net-(J1-Pad3): track 67.1 -> 0.00 mm
- net Net-(J1-Pad2): track 50.4 -> 0.00 mm
- net Net-(J1-Pad4): track 47.2 -> 0.00 mm
- net /LEFT: track 0.00 -> 43.6 mm
- net Net-(D1-Pad2): track 0.00 -> 28.8 mm
- net Net-(J1-Pad5): track 27.3 -> 0.00 mm
- net Net-(D2-Pad2): track 0.00 -> 25.9 mm
- net /UP: track 0.00 -> 25.9 mm
- net Net-(D4-Pad2): track 0.00 -> 25.7 mm
- net Net-(D3-Pad2): track 0.00 -> 25.7 mm
- net /DOWN: track 0.00 -> 23.3 mm
- net /RIGHT: track 0.00 -> 4.09 mm
- added copper zone on F.Cu, net /ROW2
- removed copper zone on B.Cu, net /ROW2
Other:
- board text added: "MX1"
- board text added: "ROW2"
- board text removed: "GND"

Commit message: Removes copper pours
Routing:
- removed copper zone on F.Cu, net /ROW2
Changed lines of the file:
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@@
-    )
-  )
-  (zone (net 5) (net_name /ROW2) (layer F.Cu) (hatch edge 0.508)
-    (connect_pads (clearance 0.508))
-    (min_thickness 0.254)
-    (fill yes (arc_segments 32) (thermal_gap 0.508) (thermal_bridge_width 0.508))
-    (polygon
-      (pts
-        (xy 171.831 72.771) (xy 173.609 76.1365) (xy 173.609 107.061) (xy 171.577 110.744) (xy 167.894 112.014)
-        (xy 101.346 112.141) (xy 97.663 110.998) (xy 96.012 109.093) (xy 95.25 106.553) (xy 95.25 76.962)
-        (xy 95.504 75.311) (xy 96.393 73.533) (xy 98.171 71.882) (xy 100.076 71.12) (xy 168.656 71.12)
-      )
     )
   )
